Commit message: livox_frame added

File: urdf/go2w_description.urdf (robot description, URDF)
Before this commit: robot go2w_description, 33 links, 32 joints
Links:
- removed link base
- added link base_footprint, mass 0
- added link base_link, mass 6.921; collision box size=0.3762 0.0935 0.114; visual mesh filename=package://go2w_description/dae/base.dae
- added link livox_frame, mass 0
Joints:
- added joint base_footprint_joint: type fixed, parent base_link, child base_footprint, origin xyz=0 0 -0.213 rpy=0 0 0, axis 0 0 0
- added joint livox_frame_joint: type fixed, parent base_link, child livox_frame, origin xyz=0.06 0 0.1 rpy=0 0 0, axis 0 0 0
- joint FL_hip_joint: parent base -> base_link
- joint FR_hip_joint: parent base -> base_link
- joint Head_upper_joint: parent base -> base_link
- joint RL_hip_joint: parent base -> base_link
- joint RR_hip_joint: parent base -> base_link
- joint imu_joint: parent base -> base_link
- joint radar_joint: parent base -> base_link
